File: sch/GridInverter.sch (EAGLE design)
At the start: 20 parts, among them Q1 IRF840, Q2 IRF840, Q3 IRF840, Q4 IRF840, Q5 IRF840, Q6 IRF840, Q7 IRF840, Q8 IRF840, Q9 IRF840

Commit message: Updated schematics, updated Readme file and an alternative SMPS algorithm
Parts:
- added C3, C4, C5, C6, C7, C8: 4.7uF, SparkFun-Capacitors:4.7UF-16V-20%,+80%-(1206)
- added D6, D7, D8, D9: 1N4004, diode:1N4004
- added IC1: 74HC00N, 74xx-eu:74HC00N
- added U1, U2, U3, U4: IRS2001SPBF, International_Rectifier_By_element14_Batch_1:IRS2001SPBF
Connections:
- net N$5 renamed LINE
- net N$8 renamed HVDC
- net N$9 renamed NEUTRAL
- removed net N$7: C1.2, D3.A, D4.A, Q5.S, Q7.S, Q9.S
- removed net O1: C2.1, L2.1, Q8.S, Q9.D
- removed net O2: C2.2, L3.1, Q6.S, Q7.D
- new net +5V: C3.1, C6.1, D6.A, D7.A, D8.A, D9.A, U1.VCC, U2.VCC, U3.VCC, U4.VCC
- new net ARD_OC1A: IC1A.I0, IC1A.I1, U1.LIN, U2.HIN
- new net ARD_OC1C: IC1B.I0, IC1B.I1, U3.LIN, U4.HIN
- new net FBR_HI_S1: Q1.G, U1.HO
- new net FBR_HI_S2: Q3.G, U2.HO
- new net FBR_LO_S1: Q2.G, U1.LO
- new net FBR_LO_S2: Q4.G, U2.LO
- new net FBR_S1: C4.1, Q1.S, Q2.D, TR1.P1, U1.VS
- new net FBR_S2: C5.2, Q3.S, Q4.D, TR1.P2, U2.VS
- new net INV_HI_S1: Q8.G, U3.HO
- new net INV_HI_S2: Q6.G, U4.HO
- new net INV_LO_S1: Q9.G, U3.LO
- new net INV_LO_S2: Q7.G, U4.LO
- new net INV_S1: C2.1, C7.1, L2.1, Q8.S, Q9.D, U3.VS
- new net INV_S2: C2.2, C8.2, L3.1, Q6.S, Q7.D, U4.VS
- new net N$11: C4.2, D6.C, U1.VB
- new net N$12: C5.1, D7.C, U2.VB
- new net NOT_ARD_OC1A: IC1A.O, U1.HIN, U2.LIN
- new net NOT_ARD_OC1C: IC1B.O, U3.HIN, U4.LIN
- net AGND: now also C1.2, C3.2, C6.2, D3.A, D4.A, Q5.S, Q7.S, Q9.S, U1.COM, U2.COM, U3.COM, U4.COM
- net N$1: now also C7.2, D8.C, U3.VB; no longer Q1.S, Q2.D, TR1.P2
- net N$2: now also C8.1, D9.C, U4.VB; no longer Q3.S, Q4.D, TR1.P1
- net S+: now also TR1.S4; no longer TR1.S3
- net S-: now also TR1.S3; no longer TR1.S4
Other:
- note added: "A"
- note added: "Booster MPPT"
- note added: "Could be same ground as SolarPanel ground?"
- note added: "Logic Signals"
- note added: "PowerCircuit"
- note removed: "Booster SMPS"
- moved on the sheet: C1, C2, D1, D2, D3, D4, D5, L1, L2, L3, Q1, Q2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
